File: keyboard.kicad_pcb (KiCad board)
At the start: 2 copper layers, 148 parts, among them J1 USB_C_Receptacle_USB2.0_16P, J2 Conn_01x02_Pin, J3 Conn_01x02_Pin, U1 STM32F072CBT6, U2 AZ1117C-3.3

Commit message: finished????!!??
Parts:
- added D63: D_Schottky, Diode_SMD:D_SOD-123F, B.Cu at (297.5, 81.0)
- added F1: Polyfuse, Fuse:Fuse_0805_2012Metric_Pad1.15x1.40mm_HandSolder, B.Cu at (292.5, 85.2)
- added H1: MountingHole, MountingHole:MountingHole_3.2mm_M3, F.Cu at (58.9, 77.6)
- added H2: MountingHole, MountingHole:MountingHole_3.2mm_M3, F.Cu at (347.6, 77.6)
- added H3: MountingHole, MountingHole:MountingHole_3.2mm_M3, F.Cu at (58.9, 175.8)
- added H4: MountingHole, MountingHole:MountingHole_3.2mm_M3, F.Cu at (347.6, 175.8)
- added U3: USBLC6-2SC6, Package_TO_SOT_SMD:SOT-23-6, B.Cu at (289.2, 85.8)
- D1, D10, D11, D12, D13, D14, D15, D16, D17, D18, D19, D2, D20, D21, D22, D23, D24, D25, D26, D27, D28, D29, D3, D30, D31, D32, D33, D34, D35, D36, D37, D38, D39, D4, D40, D41, D42, D43, D44, D45, D46, D47, D48, D49, D5, D50, D51, D52, D53, D54, D55, D56, D57, D58, D59, D6, D60, D61, D62, D7, D8, D9: footprint Diode_SMD:D_0603_1608Metric_Pad1.05x0.95mm_HandSolder -> Diode_SMD:D_SOD-123F
- moved C12 95.9 mm to (300.1, 152.8), turned to 0 degrees
- moved C5 95.6 mm to (303.9, 152.7), turned to -90 degrees
- moved C7 95.6 mm to (307.1, 148.9)
- moved C8 95.2 mm to (304.3, 140.3)
- moved U1 95.0 mm to (301.1, 146.2)
- moved C10 93.8 mm to (305.1, 135.6), turned to 180 degrees
- moved C6 93.7 mm to (294.9, 142.9)
- moved C9 93.3 mm to (300.1, 154.4), turned to 0 degrees
- moved C11 92.6 mm to (308.8, 149.3), turned to 90 degrees
- moved C3 81.0 mm to (305.3, 84.2)
- moved D27 74.9 mm to (311.2, 111.6)
- moved J3 74.8 mm to (343.8, 138.2), turned to 0 degrees
- moved D55 74.2 mm to (75.5, 169.4)
- moved D56 74.2 mm to (99.3, 169.4)
- moved D57 74.2 mm to (123.1, 169.4)
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Connections:
- J1 pad A4: +5V -> VBUS
- J1 pad A6: D+ -> D_BUS+
- J1 pad A7: D- -> D_BUS-
- J1 pad A9: +5V -> VBUS
- J1 pad B4: +5V -> VBUS
- J1 pad B6: D+ -> D_BUS+
- J1 pad B7: D- -> D_BUS-
- J1 pad B9: +5V -> VBUS
- U1 pad 10: unconnected-(U1-PA0-Pad10) -> ROW5
- U1 pad 11: unconnected-(U1-PA1-Pad11) -> COL1
- U1 pad 12: unconnected-(U1-PA2-Pad12) -> COL2
- U1 pad 13: unconnected-(U1-PA3-Pad13) -> COL3
- U1 pad 14: unconnected-(U1-PA4-Pad14) -> COL4
- U1 pad 15: unconnected-(U1-PA5-Pad15) -> COL5
- U1 pad 16: unconnected-(U1-PA6-Pad16) -> COL6
- U1 pad 17: unconnected-(U1-PA7-Pad17) -> COL7
- U1 pad 18: unconnected-(U1-PB0-Pad18) -> COL8
- U1 pad 19: unconnected-(U1-PB1-Pad19) -> COL9
- U1 pad 20: unconnected-(U1-PB2-Pad20) -> COL10
- U1 pad 21: unconnected-(U1-PB10-Pad21) -> COL11
- U1 pad 22: unconnected-(U1-PB11-Pad22) -> COL12
- U1 pad 25: unconnected-(U1-PB12-Pad25) -> ROW1
- U1 pad 26: unconnected-(U1-PB13-Pad26) -> ROW2
- U1 pad 27: unconnected-(U1-PB14-Pad27) -> ROW3
- U1 pad 28: unconnected-(U1-PB15-Pad28) -> ROW4
- U1 pad 37: unconnected-(U1-PA14-Pad37) -> COL13
- U1 pad 38: unconnected-(U1-PA15-Pad38) -> COL14
Routing:
- net COL1: track 81.1 -> 317.2 mm
- net COL2: track 98.1 -> 314.7 mm, vias 5 -> 6
- net COL3: track 99.3 -> 295.2 mm, vias 5 -> 6
- net COL4: track 75.4 -> 262.7 mm, vias 4 -> 5
- net COL5: track 74.6 -> 242.9 mm, vias 4 -> 5
- net COL6: track 73.6 -> 221.8 mm, vias 4 -> 5
- net COL7: track 99.2 -> 219.4 mm, vias 5 -> 6
- net COL8: track 74.1 -> 183.7 mm, vias 4 -> 5
- net COL9: track 74.1 -> 164.1 mm, vias 4 -> 5
- net COL10: track 73.7 -> 145.5 mm, vias 4 -> 5
- net +3.3V: track 128.8 -> 183.0 mm, vias 4 -> 3
- net ROW1: track 261.0 -> 314.1 mm, vias 0 -> 2
- net ROW4: track 247.6 -> 291.8 mm, vias 0 -> 3
- net COL11: track 97.7 -> 141.3 mm, vias 5 -> 6
- net ROW2: track 233.9 -> 271.4 mm, vias 0 -> 2
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Other:
- board outline added: 296.4 x 105.9 mm
- board text added: "3V3"
- board text added: "BOOT"
- board text added: "GND"
- board text added: "NRST"
