File: keyboard.kicad_sch (KiCad schematic)
At the start: 148 parts, among them J1 USB_C_Receptacle_USB2.0_16P, J2 Conn_01x02_Pin, J3 Conn_01x02_Pin, U1 STM32F072CBT6, U2 AZ1117C-3.3

Commit message: finished????!!??
Parts:
- added D63: D_Schottky, Diode_SMD:D_SOD-123F, symbol Device:D_Schottky
- added F1: Polyfuse, Fuse:Fuse_0805_2012Metric_Pad1.15x1.40mm_HandSolder, symbol Device:Polyfuse
- added H1, H2, H3, H4: MountingHole, MountingHole:MountingHole_3.2mm_M3, symbol Mechanical:MountingHole
- added U3: USBLC6-2SC6, Package_TO_SOT_SMD:SOT-23-6, symbol Power_Protection:USBLC6-2SC6
- D1, D10, D11, D12, D13, D14, D15, D16, D17, D18, D19, D2, D20, D21, D22, D23, D24, D25, D26, D27, D28, D29, D3, D30, D31, D32, D33, D34, D35, D36, D37, D38, D39, D4, D40, D41, D42, D43, D44, D45, D46, D47, D48, D49, D5, D50, D51, D52, D53, D54, D55, D56, D57, D58, D59, D6, D60, D61, D62, D7, D8, D9: footprint Diode_SMD:D_0603_1608Metric_Pad1.05x0.95mm_HandSolder -> Diode_SMD:D_SOD-123F
Connections:
- net +3.3V: now also D63.2 (A)
- net +5V: now also D63.1 (K), F1.2, U3.5 (VBUS); no longer J1.A4 (VBUS), J1.A9 (VBUS), J1.B4 (VBUS), J1.B9 (VBUS)
- net COL1: now also U1.11 (PA1)
- net COL10: now also U1.20 (PB2)
- net COL11: now also U1.21 (PB10)
- net COL12: now also U1.22 (PB11)
- net COL13: now also U1.37 (PA14)
- net COL14: now also U1.38 (PA15)
- net COL2: now also U1.12 (PA2)
- net COL3: now also U1.13 (PA3)
- net COL4: now also U1.14 (PA4)
- net COL5: now also U1.15 (PA5)
- net COL6: now also U1.16 (PA6)
- net COL7: now also U1.17 (PA7)
- net COL8: now also U1.18 (PB0)
- net COL9: now also U1.19 (PB1)
- net D+: now also U3.4 (I/O2); no longer J1.A6 (D+), J1.B6 (D+)
- net D-: now also U3.6 (I/O1); no longer J1.A7 (D-), J1.B7 (D-)
- net GND: now also U3.2 (GND)
- net ROW1: now also U1.25 (PB12)
- net ROW2: now also U1.26 (PB13)
- net ROW3: now also U1.27 (PB14)
- net ROW4: now also U1.28 (PB15)
- net ROW5: now also U1.10 (PA0)
- new net D_BUS+: J1.A6 (D+), J1.B6 (D+), U3.3 (I/O2)
- new net D_BUS-: J1.A7 (D-), J1.B7 (D-), U3.1 (I/O1)
- new net VBUS: F1.1, J1.A4 (VBUS), J1.A9 (VBUS), J1.B4 (VBUS), J1.B9 (VBUS)
